Commit message: update robot description to match the actual lego car size

File: description/urdf/carlikebot_description.urdf.xacro (robot description, xacro)
@@ -5,11 +5,11 @@
   <xacro:property name="PI" value="3.1415926535897931"/>
   <xacro:property name="base_mass" value="4.0" /> <!-- arbitrary value for base mass -->
-  <xacro:property name="base_width" value="0.260" />
-  <xacro:property name="base_length" value="0.525" />
-  <xacro:property name="base_height" value="0.060" />
-  <xacro:property name="wheelbase" value="0.325" />
+  <xacro:property name="base_width" value="0.19" />
+  <xacro:property name="base_length" value="0.32" />
+  <xacro:property name="base_height" value="0.045" />
+  <xacro:property name="wheelbase" value="0.24" />
   <xacro:property name="wheel_mass" value="0.34055" /> <!-- arbitrary value for wheel mass -->
-  <xacro:property name="wheel_len" value="0.045" />
-  <xacro:property name="wheel_radius" value="0.05" />
+  <xacro:property name="wheel_len" value="0.03" />
+  <xacro:property name="wheel_radius" value="0.04" />
   <!-- <xacro:property name="wheeltrack" value="" -->
   <!-- Base Link -->

Commit message: update robot base_height

File: description/urdf/carlikebot_description.urdf.xacro (robot description, xacro)
@@ -7,5 +7,5 @@
   <xacro:property name="base_width" value="0.19" />
   <xacro:property name="base_length" value="0.32" />
-  <xacro:property name="base_height" value="0.045" />
+  <xacro:property name="base_height" value="0.11" />
   <xacro:property name="wheelbase" value="0.24" />
   <xacro:property name="wheel_mass" value="0.34055" /> <!-- arbitrary value for wheel mass -->
